File: geckohat.kicad_pcb (KiCad board)
At the start: 2 copper layers, 65 x 56 mm, 19 parts, among them J1 CONN_02X20, U1 EFM32JG1B100F128GM32, U2 LP2985LV

Commit message: Updates
Parts:
- added JP1: tie, Resistors_SMD:R_0603, F.Cu at (123.0, 90.0)
- added JP2: tie, Resistors_SMD:R_0603, F.Cu at (125.0, 90.0)
- added JP3: tie, Resistors_SMD:R_0603, F.Cu at (127.0, 90.0)
- added JP4: tie, Resistors_SMD:R_0603, F.Cu at (129.0, 90.0)
- added JP5: tie, Resistors_SMD:R_0603, F.Cu at (131.0, 90.0)
- added REF**: hole_2.75, holes:hole_2.75, F.Cu at (124.7, 74.9)
- added REF**: hole_2.75, holes:hole_2.75, F.Cu at (182.7, 74.9)
- added REF**: hole_2.75, holes:hole_2.75, F.Cu at (124.7, 123.9)
- added REF**: hole_2.75, holes:hole_2.75, F.Cu at (182.7, 123.9)
- added RN3: CAY16-221J4LF, Resistors_SMD:R_Array_Convex_4x0603, F.Cu at (149.9, 80.0)
- added RN4: CAY16-221J4LF, Resistors_SMD:R_Array_Convex_4x0603, F.Cu at (156.6, 79.9)
- added RN5: CAY16-221J4LF, Resistors_SMD:R_Array_Convex_4x0603, F.Cu at (163.5, 81.2)
- added RN6: CAY16-221J4LF, Resistors_SMD:R_Array_Convex_4x0603, F.Cu at (171.1, 81.2)
- added RN7: CAY16-221J4LF, Resistors_SMD:R_Array_Convex_4x0603, F.Cu at (174.9, 79.9)
- RN1, RN2: value R_Pack04 -> CAY16-221J4LF
- moved C1 65.6 mm to (124.0, 79.0), turned to 180 degrees
- moved C4 63.2 mm to (115.0, 87.5)
- moved C5 59.4 mm to (124.0, 86.0)
- moved C3 55.0 mm to (127.0, 85.0), turned to 270 degrees
- moved C6 48.8 mm to (126.5, 97.0), turned to 90 degrees
- moved C9 48.0 mm to (128.0, 97.0), turned to 90 degrees
- moved C2 47.2 mm to (129.5, 97.0), turned to 90 degrees
- moved C8 45.4 mm to (122.5, 104.5), turned to 270 degrees
- moved C7 41.4 mm to (131.5, 102.5), turned to 270 degrees
- moved R2 41.2 mm to (123.0, 110.0), turned to 90 degrees
- moved R1 39.7 mm to (125.0, 110.0), turned to 90 degrees
- moved R3 38.3 mm to (127.0, 110.0), turned to 90 degrees
- moved U1 2.77 mm to (127.0, 102.5)
- moved U2 2.53 mm to (124.0, 82.5), turned to 270 degrees
- moved D1 2.18 mm to (125.0, 116.0), turned to 270 degrees
- renumbered REF** to PA1
Connections:
- net Net-(J1-Pad13) renamed /GPIO27
- net Net-(J1-Pad3) renamed /GPIO2
- net Net-(J1-Pad5) renamed /GPIO3
- net Net-(J1-Pad7) renamed /GPIO4
- J1 pad 11: Net-(J1-Pad11) -> /GPIO17
- J1 pad 15: (no net) -> /GPIO22
- J1 pad 16: (no net) -> /GPIO23
- J1 pad 18: (no net) -> /GPIO24
- J1 pad 19: (no net) -> /GPIO10
- J1 pad 21: (no net) -> /GPIO9
- J1 pad 22: (no net) -> /GPIO25
- J1 pad 23: (no net) -> /GPIO11
- J1 pad 24: (no net) -> /GPIO8
- J1 pad 26: (no net) -> /GPIO7
- J1 pad 27: (no net) -> /ID_SD
- J1 pad 28: (no net) -> /ID_SC
- J1 pad 29: (no net) -> /GPIO5
- J1 pad 31: (no net) -> /GPIO6
- J1 pad 32: (no net) -> /GPIO12
- J1 pad 33: (no net) -> /GPIO13
- J1 pad 35: (no net) -> /GPIO19
- J1 pad 36: (no net) -> /GPIO16
- J1 pad 37: (no net) -> /GPIO26
- J1 pad 38: (no net) -> /GPIO20
- J1 pad 39: (no net) -> GND
- J1 pad 40: (no net) -> /GPIO21
- PA1 pad 1: (no net) -> VDD
- PA1 pad 10: (no net) -> /PGPIO15
- PA1 pad 11: (no net) -> /PGPIO17
- PA1 pad 12: (no net) -> /PGPIO18
- PA1 pad 13: (no net) -> /PGPIO27
- PA1 pad 14: (no net) -> GND
- PA1 pad 15: (no net) -> /PGPIO22
- PA1 pad 16: (no net) -> /PGPIO23
- PA1 pad 17: (no net) -> VDD
- PA1 pad 18: (no net) -> /PGPIO24
- PA1 pad 19: (no net) -> /PGPIO10
- PA1 pad 2: (no net) -> +5V
- PA1 pad 20: (no net) -> GND
- PA1 pad 21: (no net) -> /PGPIO9
- PA1 pad 22: (no net) -> /PGPIO25
- PA1 pad 23: (no net) -> /PGPIO11
- PA1 pad 24: (no net) -> /PGPIO8
- PA1 pad 25: (no net) -> GND
- PA1 pad 26: (no net) -> /PGPIO7
- PA1 pad 27: (no net) -> /PID_SD
- PA1 pad 28: (no net) -> /PID_SC
- PA1 pad 29: (no net) -> /PGPIO5
- PA1 pad 3: (no net) -> /PGPIO2
- PA1 pad 30: (no net) -> GND
- PA1 pad 31: (no net) -> /PGPIO6
- PA1 pad 32: (no net) -> /PGPIO12
- PA1 pad 33: (no net) -> /PGPIO13
- PA1 pad 34: (no net) -> GND
- PA1 pad 35: (no net) -> /PGPIO19
- PA1 pad 36: (no net) -> /PGPIO16
- PA1 pad 37: (no net) -> /PGPIO26
- PA1 pad 38: (no net) -> /PGPIO20
- PA1 pad 39: (no net) -> GND
- PA1 pad 4: (no net) -> +5V
- PA1 pad 40: (no net) -> /PGPIO21
- PA1 pad 5: (no net) -> /PGPIO3
- PA1 pad 6: (no net) -> GND
- PA1 pad 7: (no net) -> /PGPIO4
- PA1 pad 8: (no net) -> /PGPIO14
- PA1 pad 9: (no net) -> GND
- RN1 pad 1: (no net) -> /PGPIO2
- RN1 pad 2: (no net) -> /PGPIO3
- RN1 pad 3: (no net) -> /PGPIO4
- RN1 pad 4: /RPI_TX -> /PGPIO14
- RN2 pad 1: /RPI_RX -> /PGPIO15
- RN2 pad 2: /nRST -> /PGPIO17
- RN2 pad 3: (no net) -> /PGPIO18
- RN2 pad 4: (no net) -> /PGPIO27
- RN2 pad 6: Net-(J1-Pad11) -> /GPIO18
- RN2 pad 7: /GPIO18 -> /GPIO17
- U1 pad 1: (no net) -> /SWD_CLK
- U1 pad 10: (no net) -> /PROT1
- U1 pad 11: (no net) -> /PROT2
- U1 pad 12: (no net) -> /PROT3
- U1 pad 13: (no net) -> /PROT4
- U1 pad 14: (no net) -> /PROT5
- U1 pad 15: (no net) -> /PROT6
- U1 pad 16: (no net) -> /PROT7
- U1 pad 2: (no net) -> /SWD_IO
Routing:
- net Net-(J1-Pad11): track 6.19 -> 0.00 mm
- net /GPIO18: track 3.08 -> 7.16 mm
- net /GPIO17: track 0.00 -> 2.10 mm
Other:
- outline, holes or cut-outs redrawn
- net class Default: via_drill 0.3 -> 0.2
- rule pad_to_mask_clearance: 0.2 -> 0.1
- rule via_min_drill: 0.3 -> 0.2

Commit message: Updates
Parts:
- U1: footprint Housings_DFN_QFN:QFN-32-1EP_5x5mm_Pitch0.5mm -> qfn:QFN-32-1EP_5x5mm_Pitch0.5mm
Routing:
- net /PGPIO25: track 0.00 -> 35.7 mm
- net /PGPIO24: track 0.00 -> 28.6 mm
- net /PGPIO18: track 0.00 -> 18.8 mm
- net /PGPIO14: track 0.00 -> 17.6 mm
- net /PGPIO15: track 0.00 -> 15.9 mm
- net /GPIO18: track 7.16 -> 0.00 mm
- net VDD: track 0.00 -> 5.57 mm
- net Net-(C9-Pad1): track 0.00 -> 2.25 mm
- net /GPIO17: track 2.10 -> 0.00 mm
Other:
- net class Default: via_dia 0.9 -> 0.6
- rule via_min_size: 0.9 -> 0.6

Commit message: Updates
Parts:
- added J2: TEST_1P, Wire_Pads:SolderWirePad_single_1mmDrill, F.Cu at (123.0, 98.0)
- added Y1: 38.4 MHz, Crystals:Crystal_SMD_SeikoEpson_FA238-4pin_3.2x2.5mm_HandSoldering, F.Cu at (124.0, 106.0)
- added Y2: 32kHz, Crystals:Crystal_C26-LF_d2.1mm_l6.5mm_Vertical, F.Cu at (131.5, 98.4)
- D1: value LED_ARGB -> LED_RGB; footprint LEDs:LED_WS2812-PLCC6 -> led:LED_RGB_5050+PLCC4
- U1: footprint qfn:QFN-32-1EP_5x5mm_Pitch0.5mm -> qfn:QFN-32-handsolder
- moved C4 17.2 mm to (130.5, 80.0)
- moved R3 4.61 mm to (122.5, 111.0)
- moved C2 3.81 mm to (131.0, 93.5)
- moved C6 3.81 mm to (128.0, 93.5)
- moved C9 3.81 mm to (129.5, 93.5)
- moved C8 3.50 mm to (122.5, 101.0)
- moved U1 3.50 mm to (127.0, 99.0)
- moved RN1 3.38 mm to (138.0, 80.0)
- moved RN6 3.31 mm to (168.0, 80.0), turned to 90 degrees
- moved RN5 2.74 mm to (161.0, 80.0), turned to 90 degrees
- moved RN7 2.39 mm to (172.5, 80.0), turned to 90 degrees
- moved JP5 2.00 mm to (129.0, 90.0)
- moved JP4 1.50 mm to (127.5, 90.0)
- moved R2 1.41 mm to (124.0, 111.0)
- moved RN3 1.36 mm to (148.5, 80.0)
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Connections:
- D1 pad 1: VDD -> Net-(D1-Pad1)
- D1 pad 4: Net-(D1-Pad4) -> VDD
- D1 pad 5: (no net) -> VDD
- D1 pad 6: (no net) -> VDD
- PA1 pad A10: (no net) -> /PROT10
- PA1 pad A11: (no net) -> /PROT11
- PA1 pad A12: (no net) -> /PROT12
- PA1 pad A13: (no net) -> /PROT13
- PA1 pad A14: (no net) -> /PROT14
- PA1 pad A8: (no net) -> /PROT8
- PA1 pad A9: (no net) -> /PROT9
- PA1 pad GND: (no net) -> GND
- R1 pad 1: Net-(D1-Pad2) -> Net-(D1-Pad1)
- R2 pad 1: Net-(D1-Pad3) -> Net-(D1-Pad2)
- R3 pad 1: Net-(D1-Pad4) -> Net-(D1-Pad3)
- U1 pad 10: /PROT1 -> /PROT14
- U1 pad 11: /PROT2 -> /PROT13
- U1 pad 12: /PROT3 -> /PROT12
- U1 pad 13: /PROT4 -> /PROT11
- U1 pad 14: /PROT5 -> /PROT10
- U1 pad 15: /PROT6 -> /PROT9
- U1 pad 16: /PROT7 -> /PROT8
- U1 pad 17: (no net) -> /PROT7
- U1 pad 18: (no net) -> /PROT6
- U1 pad 23: (no net) -> Net-(U1-Pad23)
- U1 pad 24: (no net) -> Net-(U1-Pad24)
- U1 pad 28: (no net) -> /PROT5
- U1 pad 29: (no net) -> /PROT4
- U1 pad 3: (no net) -> /SWD_SWO
- U1 pad 30: (no net) -> /PROT3
- U1 pad 31: (no net) -> /PROT2
- U1 pad 32: (no net) -> /PROT1
- U1 pad 7: (no net) -> Net-(U1-Pad7)
- U1 pad 8: (no net) -> Net-(U1-Pad8)
Routing:
- net VDD: track 5.57 -> 139.6 mm, vias 0 -> 5
- net +5V: track 0.00 -> 33.8 mm
- net /PROT14: track 0.00 -> 22.5 mm
- net /PROT13: track 0.00 -> 19.8 mm
- net /LED_G: track 0.00 -> 18.3 mm, vias 0 -> 2
- net /LED_B: track 0.00 -> 17.9 mm, vias 0 -> 2
- net /PROT5: track 0.00 -> 17.5 mm, vias 0 -> 1
- net /LED_R: track 0.00 -> 17.3 mm, vias 0 -> 2
- net /nRST: track 0.00 -> 17.1 mm, vias 0 -> 2
- net /PROT12: track 0.00 -> 17.0 mm
- net /PROT4: track 0.00 -> 16.0 mm, vias 0 -> 1
- net /PROT1: track 0.00 -> 15.4 mm, vias 0 -> 1
- net /PROT6: track 0.00 -> 14.9 mm
- net /PROT3: track 0.00 -> 14.7 mm, vias 0 -> 1
- net /PROT2: track 0.00 -> 14.3 mm, vias 0 -> 1
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- added copper zone on B.Cu, net GND
- added copper zone on F.Cu, net GND
Other:
- net class Big supply added: clearance 0.16, trace_width 0.3, via_dia 1, via_drill 0.4
- net class Supply added: clearance 0.16, trace_width 0.2, via_dia 0.7, via_drill 0.3
- board text added: "1"
- board text added: "10"
- board text added: "2"
- board text added: "3"
- board text added: "7"
- board text added: "8"
- board text added: "9"

Commit message: DRC fixes and stuff
Parts:
- moved C1 0.50 mm to (124.5, 79.0)
Routing:
- net GND: track 8.75 -> 57.9 mm, vias 8 -> 12
- net +5V: track 33.8 -> 30.8 mm
- net /SWD_IO: track 10.00 -> 10.6 mm

Commit message: Net ties
Parts:
- JP1, JP2, JP3, JP4, JP5: footprint Resistors_SMD:R_0603 -> tie:tie_0603
Other:
- board text added: "RST"
- board text added: "RX"
- board text added: "SCLK"
- board text added: "SIO"
- board text added: "TX"
