File: geckohat.sch (KiCad schematic (older format))
At the start: 22 parts, among them J1 CONN_02X20, U1 EFM32JG1B100F128GM32, U2 LP2985LV, Y1 40 MHz, Y2 32kHz

Commit message: Updates
Parts:
- added JP1, JP2, JP3, JP4, JP5: tie, symbol Jumper_NC_Small
- added PA1: protoarea, symbol protoarea
- added RN5, RN6, RN7: CAY16-221J4LF, Resistors_SMD:R_Array_Convex_4x0603, symbol R_Pack04
Connections:
- net labels added: GPIO10, GPIO11, GPIO12, GPIO13, GPIO16, GPIO17, GPIO19, GPIO2, GPIO20, GPIO21, GPIO22, GPIO23, GPIO26, GPIO27, GPIO3, GPIO4, GPIO5, GPIO6, GPIO9, ID_SC, ID_SD, PGPIO10, PGPIO11, PGPIO12, PGPIO13, PGPIO14, PGPIO15, PGPIO16, PGPIO17, PGPIO18, PGPIO19, PGPIO2, PGPIO20, PGPIO21, PGPIO22, PGPIO23, PGPIO24, PGPIO25, PGPIO26, PGPIO27, PGPIO3, PGPIO4, PGPIO5, PGPIO6, PGPIO7, PGPIO8, PGPIO9, PID_SC, PID_SD, PROT1, PROT2, PROT3, PROT4, PROT5, PROT6, PROT7
- net labels removed: +3.3V
- wire segments 103 -> 200
- no-connect marks 0 -> 2
Other:
- note added: "RXD0"
- note added: "SPI"
- note added: "SPI_CE0"
- note added: "SPI_CE1"
- note added: "TXD0"
- moved on the sheet: C9, D1, J1, R1, R2, R3, RN1, RN2, RN3, RN4, U1, Y1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

Commit message: Updates
Parts:
- JP1, JP2, JP3, JP4, JP5: footprint (none) -> Resistors_SMD:R_0603
- PA1: footprint (none) -> protoarea:protoarea

Commit message: Updates
Parts:
- removed D1: LED_ARGB, LEDs:LED_WS2812-PLCC6, symbol LED_ARGB
- removed Y1: 40 MHz, symbol Crystal_Small
- added D?: LED_RGB, symbol LED_RGB
- added J2: TEST_1P, Wire_Pads:SolderWirePad_single_1mmDrill, symbol TEST_1P
- added Y1: 38.4 MHz, Crystals:Crystal_SMD_SeikoEpson_FA238-4pin_3.2x2.5mm_HandSoldering, symbol Crystal_GND24
- U1: footprint Housings_DFN_QFN:QFN-32-1EP_5x5mm_Pitch0.5mm -> qfn:QFN-32-handsolder
- Y2: footprint (none) -> Crystals:Crystal_C26-LF_d2.1mm_l6.5mm_Vertical
Connections:
- net GND: now also PA1.GND, Y1.2, Y1.4
- net PROT1: now also U1.32 (PC11); no longer U1.10 (PD9)
- net PROT2: now also U1.31 (PC10); no longer U1.11 (PD10)
- net PROT3: now also U1.30 (PC9); no longer U1.12 (PD11)
- net PROT4: now also U1.29 (PC8); no longer U1.13 (PD12)
- net PROT5: now also U1.28 (PC7); no longer U1.14 (PD13)
- net PROT6: now also U1.18 (PA1); no longer U1.15 (PD14)
- net PROT7: now also U1.17 (PA0); no longer U1.16 (PD15)
- net VDD: now also PA1.VCC, D?.4 (BA), D?.5 (GA), D?.6 (RA)
- net at U1.7 (HFXTAL_N): now also Y1.3
- net at U1.8 (HFXTAL_P): now also Y1.1
- net at R1.1: now also D?.1 (RK)
- net at R2.1: now also D?.2 (GK)
- net at R3.1: now also D?.3 (BK)
- net SWD_SWO: now reaches U1.3 (PF2)
- net SWD_SWO: now also J2.1
- net PROT10: now reaches PA1.A10
- net PROT10: now also U1.14 (PD13)
- net PROT11: now reaches PA1.A11
- net PROT11: now also U1.13 (PD12)
- net PROT12: now reaches PA1.A12
- net PROT12: now also U1.12 (PD11)
- net PROT13: now reaches PA1.A13
- net PROT13: now also U1.11 (PD10)
- net PROT14: now reaches PA1.A14
- net PROT14: now also U1.10 (PD9)
- net PROT8: now reaches PA1.A8
- net PROT8: now also U1.16 (PD15)
- net PROT9: now reaches PA1.A9
- net PROT9: now also U1.15 (PD14)
Other:
- note added: "U2: AP2210K-3.3, alt: NJM2866F33-TE1, alt: LP2985\nOption: change VREG for 1.8V operation?\nResistor net: Bourns CAY16-221J4LF, is 3.2×1.6 mm\nCrystal: TSX-3225 38.4000MF10Z-AS3\nFIXME:\n - Add ARM debug header\n - Connect RPi serial port"
- note removed: "U2: AP2210K-3.3, alt: NJM2866F33-TE1, alt: LP2985\nOption: change VREG for 1.8V operation?\nResistor net: Bourns CAY16-221J4LF, is 3.2×1.6 mm\nFIXME:\n - Add ARM debug header\n - Connect RPi serial port"
Changed lines of the file:
@@
-$EndComp
-$Comp
-L Crystal_Small Y1
-U 1 1 59809C18
-P 1100 4850
-F 0 "Y1" H 1100 4950 50  0000 C CNN
-F 1 "40 MHz" H 1100 4750 50  0000 C CNN
-F 2 "" H 1100 4850 50  0001 C CNN
-F 3 "" H 1100 4850 50  0001 C CNN
-	1    1100 4850
-	0    1    1    0
 $EndComp
 $Comp
@@
 F 0 "Y2" H 3900 4350 50  0000 C CNN
 F 1 "32kHz" H 3900 4150 50  0000 C CNN
-F 2 "" H 3900 4250 50  0001 C CNN
+F 2 "Crystals:Crystal_C26-LF_d2.1mm_l6.5mm_Vertical" H 3900 4250 50  0001 C CNN
 F 3 "" H 3900 4250 50  0001 C CNN
 	1    3900 4250
@@
 $EndComp
 Text Notes 3750 6700 0    60   ~ 0
-U2: AP2210K-3.3, alt: NJM2866F33-TE1, alt: LP2985\nOption: change VREG for 1.8V operation?\nResistor net: Bourns CAY16-221J4LF, is 3.2×1.6 mm\nFIXME:\n  - Add ARM debug header\n  - Connect RPi serial port
+U2: AP2210K-3.3, alt: NJM2866F33-TE1, alt: LP2985\nOption: change VREG for 1.8V operation?\nResistor net: Bourns CAY16-221J4LF, is 3.2×1.6 mm\nCrystal:  TSX-3225 38.4000MF10Z-AS3\nFIXME:\n  - Add ARM debug header\n  - Connect RPi serial port
 $Comp
 L +5V #PWR011
@@
 	1    0    0    -1
 $EndComp
-$Comp
-L LED_ARGB D1
-U 1 1 5980C2E6
-P 4700 4600
-F 0 "D1" H 4700 4970 50  0000 C CNN
-F 1 "LED_ARGB" H 4700 4250 50  0000 C CNN
-F 2 "LEDs:LED_WS2812-PLCC6" H 4700 4550 50  0001 C CNN
-F 3 "" H 4700 4550 50  0001 C CNN
-	1    4700 4600
-	1    0    0    -1
-$EndComp
 Text Label 7850 2450 3    60   ~ 0
 GPIO14
@@
 F 0 "U1" H 3150 3850 60  0000 C CNN
 F 1 "EFM32JG1B100F128GM32" H 2550 4550 39  0000 C CNN
-F 2 "Housings_DFN_QFN:QFN-32-1EP_5x5mm_Pitch0.5mm" H 2200 4700 60  0001 C CNN
+F 2 "qfn:QFN-32-handsolder" H 2200 4700 60  0001 C CNN
 F 3 "" H 2200 4700 60  0001 C CNN
 	1    2550 4550
@@
 	1200 4800 1700 4800
 Wire Wire Line
-	1200 4800 1200 4750
-Wire Wire Line
-	1200 4750 1100 4750
-Wire Wire Line
 	1200 4900 1700 4900
-Wire Wire Line
-	1200 4900 1200 4950
-Wire Wire Line
-	1200 4950 1100 4950
 Wire Wire Line
 	1150 4100 1700 4100
@@
 Wire Wire Line
 	2900 5800 2900 5400
+Text Label 2200 3300 3    60   ~ 0
+PROT1
+Text Label 2300 3300 3    60   ~ 0
+PROT2
+Text Label 2400 3300 3    60   ~ 0
+PROT3
+Text Label 2500 3300 3    60   ~ 0
+PROT4
+Text Label 2600 3300 3    60   ~ 0
+PROT5
+Text Label 3800 4800 2    60   ~ 0
+PROT6
+Text Label 3800 4900 2    60   ~ 0
+PROT7
+$Comp
+L GND #PWR044
+U 1 1 59844406
+P 10000 6100
+F 0 "#PWR044" H 10000 5850 50  0001 C CNN
+F 1 "GND" H 10000 5950 50  0000 C CNN
+F 2 "" H 10000 6100 50  0001 C CNN
+F 3 "" H 10000 6100 50  0001 C CNN
+	1    10000 6100
+	1    0    0    -1
+$EndComp
+$Comp
+L VDD #PWR045
+U 1 1 598445C3
+P 10250 5850
+F 0 "#PWR045" H 10250 5700 50  0001 C CNN
+F 1 "VDD" H 10250 6000 50  0000 C CNN
+F 2 "" H 10250 5850 50  0001 C CNN
+F 3 "" H 10250 5850 50  0001 C CNN
+	1    10250 5850
+	1    0    0    -1
+$EndComp
+Wire Wire Line
+	10000 5900 10000 6100
+Wire Wire Line
+	10100 5900 10100 6050
+Wire Wire Line
+	10100 6050 10250 6050
+Wire Wire Line
+	10250 6050 10250 5850
+Wire Wire Line
+	2600 3700 2600 3300
+Wire Wire Line
+	2500 3700 2500 3300
+Wire Wire Line
+	2400 3700 2400 3300
+Wire Wire Line
+	2300 3700 2300 3300
+Wire Wire Line
+	2200 3700 2200 3300
+Text Label 2900 5800 1    60   ~ 0
+PROT8
+Text Label 2800 5800 1    60   ~ 0
+PROT9
+Text Label 2700 5800 1    60   ~ 0
+PROT10
+Text Label 2600 5800 1    60   ~ 0
+PROT11
+Text Label 2500 5800 1    60   ~ 0
+PROT12
+Wire Wire Line
+	1700 4400 1350 4400
+Text Label 1350 4400 0    60   ~ 0
+SWD_SWO
+Wire Wire Line
+	3400 4800 3800 4800
+Wire Wire Line
+	3400 4900 3800 4900
+Text Label 2400 5800 1    60   ~ 0
+PROT13
 Text Label 2300 5800 1    60   ~ 0
-PROT1
-Text Label 2400 5800 1    60   ~ 0
-PROT2
-Text Label 2500 5800 1    60   ~ 0
-PROT3
-Text Label 2600 5800 1    60   ~ 0
-PROT4
-Text Label 2700 5800 1    60   ~ 0
-PROT5
-Text Label 2800 5800 1    60   ~ 0
-PROT6
-Text Label 2900 5800 1    60   ~ 0
-PROT7
+PROT14
+$Comp
+L TEST_1P J2
+U 1 1 59847B90
+P 1350 4400
+F 0 "J2" H 1350 4670 50  0000 C CNN
+F 1 "TEST_1P" H 1350 4600 50  0000 C CNN
+F 2 "Wire_Pads:SolderWirePad_single_1mmDrill" H 1550 4400 50  0001 C CNN
+F 3 "" H 1550 4400 50  0001 C CNN
+	1    1350 4400
+	0    -1   -1   0
+$EndComp
+Wire Wire Line
+	9100 6400 9100 5900
+Wire Wire Line
+	9200 6400 9200 5900
+Wire Wire Line
+	9300 6400 9300 5900
+Wire Wire Line
+	9400 6400 9400 5900
+Wire Wire Line
+	9500 6400 9500 5900
+Wire Wire Line
+	9600 6400 9600 5900
+Wire Wire Line
+	9700 6400 9700 5900
+Text Label 9100 6400 1    60   ~ 0
+PROT8
+Text Label 9200 6400 1    60   ~ 0
+PROT9
+Text Label 9300 6400 1    60   ~ 0
+PROT10
+Text Label 9400 6400 1    60   ~ 0
+PROT11
+Text Label 9500 6400 1    60   ~ 0
+PROT12
+Text Label 9600 6400 1    60   ~ 0
+PROT13
+Text Label 9700 6400 1    60   ~ 0
+PROT14
+Wire Wire Line
+	1200 4800 1200 4700
+Wire Wire Line
+	1200 4700 900  4700
+Wire Wire Line
+	1200 4900 1200 5000
+Wire Wire Line
+	1200 5000 900  5000
+Wire Wire Line
+	1100 4850 1100 5100
+Wire Wire Line
+	1100 5100 700  5100
+Wire Wire Line
+	700  4850 700  5200
+Connection ~ 700  5100
+$Comp
+L GND #PWR046
+U 1 1 5984A03E
+P 700 5200
+F 0 "#PWR046" H 700 4950 50  0001 C CNN
+F 1 "GND" H 700 5050 50  0000 C CNN
+F 2 "" H 700 5200 50  0001 C CNN
+F 3 "" H 700 5200 50  0001 C CNN
+	1    700  5200
+	1    0    0    -1
+$EndComp
+$Comp
+L Crystal_GND24 Y1
+U 1 1 5984A564
+P 900 4850
+F 0 "Y1" H 1025 5050 50  0000 L CNN
+F 1 "38.4 MHz" H 1025 4975 50  0000 L CNN
+F 2 "Crystals:Crystal_SMD_SeikoEpson_FA238-4pin_3.2x2.5mm_HandSoldering" H 900 4850 50  0001 C CNN
+F 3 "" H 900 4850 50  0001 C CNN
+	1    900  4850
+	0    -1   -1   0
+$EndComp
+$Comp
+L LED_RGB D?
+U 1 1 5984CA47
+P 4700 4600
+F 0 "D?" H 4700 4970 50  0000 C CNN
+F 1 "LED_RGB" H 4700 4250 50  0000 C CNN
+F 2 "" H 4700 4550 50  0001 C CNN
+F 3 "" H 4700 4550 50  0001 C CNN
+	1    4700 4600
+	1    0    0    -1
+$EndComp
+Wire Wire Line
+	4900 4400 4900 4800
+Connection ~ 4900 4600
 $EndSCHEMATC

Commit message: DRC fixes and stuff
Parts:
- D1: renamed from D?; footprint (none) -> led:LED_RGB_5050+PLCC4
Changed lines of the file:
@@
 $EndComp
 $Comp
-L LED_RGB D?
+L LED_RGB D1
 U 1 1 5984CA47
 P 4700 4600
-F 0 "D?" H 4700 4970 50  0000 C CNN
+F 0 "D1" H 4700 4970 50  0000 C CNN
 F 1 "LED_RGB" H 4700 4250 50  0000 C CNN
-F 2 "" H 4700 4550 50  0001 C CNN
+F 2 "led:LED_RGB_5050+PLCC4" H 4700 4550 50  0001 C CNN
 F 3 "" H 4700 4550 50  0001 C CNN
 	1    4700 4600

Commit message: Net ties
Parts:
- JP1, JP2, JP3, JP4, JP5: footprint Resistors_SMD:R_0603 -> tie:tie_0603
Changed lines of the file:
@@
 F 0 "JP1" H 7850 3730 50  0000 C CNN
 F 1 "tie" H 7860 3590 50  0001 C CNN
-F 2 "Resistors_SMD:R_0603" H 7850 3650 50  0001 C CNN
+F 2 "tie:tie_0603" H 7850 3650 50  0001 C CNN
 F 3 "" H 7850 3650 50  0001 C CNN
 	1    7850 3650
@@
 F 0 "JP3" H 8250 3730 50  0000 C CNN
 F 1 "tie" H 8260 3590 50  0001 C CNN
-F 2 "Resistors_SMD:R_0603" H 8250 3650 50  0001 C CNN
+F 2 "tie:tie_0603" H 8250 3650 50  0001 C CNN
 F 3 "" H 8250 3650 50  0001 C CNN
 	1    8250 3650
@@
 F 0 "JP4" H 8750 3730 50  0000 C CNN
 F 1 "tie" H 8760 3590 50  0001 C CNN
-F 2 "Resistors_SMD:R_0603" H 8750 3650 50  0001 C CNN
+F 2 "tie:tie_0603" H 8750 3650 50  0001 C CNN
 F 3 "" H 8750 3650 50  0001 C CNN
 	1    8750 3650
@@
 F 0 "JP5" H 9150 3730 50  0000 C CNN
 F 1 "tie" H 9160 3590 50  0001 C CNN
-F 2 "Resistors_SMD:R_0603" H 9150 3650 50  0001 C CNN
+F 2 "tie:tie_0603" H 9150 3650 50  0001 C CNN
 F 3 "" H 9150 3650 50  0001 C CNN
 	1    9150 3650
@@
 F 0 "JP2" H 8050 3730 50  0000 C CNN
 F 1 "tie" H 8060 3590 50  0001 C CNN
-F 2 "Resistors_SMD:R_0603" H 8050 3650 50  0001 C CNN
+F 2 "tie:tie_0603" H 8050 3650 50  0001 C CNN
 F 3 "" H 8050 3650 50  0001 C CNN
 	1    8050 3650
