File: geckohat.sch (KiCad schematic (older format))
At the start: 32 parts, among them J1 CONN_02X20, J2 TEST_1P, U1 EFM32JG1B100F128GM32, U2 LP2985LV, Y1 38.4 MHz, Y2 32kHz

Commit message: Unknown changes that were lying around
Other:
- note added: "U2: AP2210K-3.3, alt: NJM2866F33-TE1, alt: LP2985\nOption: change VREG for 1.8V operation?\nResistor net: Bourns CAY16-221J4LF, is 3.2×1.6 mm\nCrystal: TSX-3225 38.4000MF10Z-AS3\nFIXME:\n - Add ARM debug header\n - reset switch option\n - Elemental logo\n - OSHW logo\n - Revision info on bottom side\n - Jumpers over resistor nets\n - 3V3 vreg bypass jumper\n - Isolate GND on bottom of U1 and add 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"
- note removed: "U2: AP2210K-3.3, alt: NJM2866F33-TE1, alt: LP2985\nOption: change VREG for 1.8V operation?\nResistor net: Bourns CAY16-221J4LF, is 3.2×1.6 mm\nCrystal: TSX-3225 38.4000MF10Z-AS3\nFIXME:\n - Add ARM debug header\n - reset switch option\n - Elemental logo\n - OSHW logo\n - Revision info on bottom side\n - Jumpers over resistor nets\n - 3V3 vreg bypass jumper"
Changed lines of the file:
@@
 $EndComp
 Text Notes 3750 6700 0    60   ~ 0
-U2: AP2210K-3.3, alt: NJM2866F33-TE1, alt: LP2985\nOption: change VREG for 1.8V operation?\nResistor net: Bourns CAY16-221J4LF, is 3.2×1.6 mm\nCrystal:  TSX-3225 38.4000MF10Z-AS3\nFIXME:\n  - Add ARM debug header\n  - reset switch option\n  - Elemental logo\n  - OSHW logo\n  - Revision info on bottom side\n  - Jumpers over resistor nets\n  - 3V3 vreg bypass jumper
+U2: AP2210K-3.3, alt: NJM2866F33-TE1, alt: LP2985\nOption: change VREG for 1.8V operation?\nResistor net: Bourns CAY16-221J4LF, is 3.2×1.6 mm\nCrystal:  TSX-3225 38.4000MF10Z-AS3\nFIXME:\n  - Add ARM debug header\n  - reset switch option\n  - Elemental logo\n  - OSHW logo\n  - Revision info on bottom side\n  - Jumpers over resistor nets\n  - 3V3 vreg bypass jumper\n  - Isolate GND on bottom of U1 and add thermals, for solderability
 $Comp
 L +5V #PWR011

Commit message: Work on board: fix header rotation, LED, use discreet resistors
Parts:
- removed D1: LED_RGB, led:LED_RGB_5050+PLCC4, symbol LED_RGB
- removed RN1, RN2, RN3, RN4, RN5, RN6, RN7: CAY16-221J4LF, Resistors_SMD:R_Array_Convex_4x0603, symbol R_Pack04
- added D1: LED_ARGB, led:LED_Avago_PLCC4_3.2x2.8mm_CW, symbol LED_ARGB
- added JP6: tie, tie:tie_0603, symbol Jumper_NC_Small
- added JP7: Jumper_NO_Small, tie:tie_0603_open, symbol Jumper_NO_Small
- added R10, R11, R12, R13, R14, R15, R16, R17, R18, R19, R20, R21, R22, R23, R24, R25, R26, R27, R28, R29, R30, R31, R4, R5, R6, R7, R8, R9: R, r_local:R_0603_1608Metric_Pad0.84x1.00mm_HandSolder, symbol R
- added R32, R33: 3k9, r_local:R_0603_1608Metric_Pad0.84x1.00mm_HandSolder, symbol R_Small
- added U3: CAT24C32, Housings_SOIC:SOIC-8_3.9x4.9mm_Pitch1.27mm, symbol 24LC04
- C4: footprint Capacitors_SMD:C_1206_HandSoldering -> c_local:C_1206_3216Metric_Pad1.24x1.80mm_HandSolder
- R1, R2, R3: footprint Resistors_SMD:R_0603_HandSoldering -> r_local:R_0603_1608Metric_Pad0.84x1.00mm_HandSolder
Connections:
- net GND: now also U3.1 (A0), U3.2 (A1), U3.3 (A2), U3.4 (GND)
- net GPIO10: now also R15.1
- net GPIO11: now also R18.1
- net GPIO12: now also R25.1
- net GPIO13: now also R26.1
- net GPIO14: now also R7.1
- net GPIO15: now also R8.1
- net GPIO16: now also R28.1
- net GPIO17: now also R9.1
- net GPIO18: now also R10.1
- net GPIO19: now also R27.1
- net GPIO2: now also R4.1
- net GPIO20: now also R30.1
- net GPIO21: now also R31.1
- net GPIO22: now also R12.1
- net GPIO23: now also R13.1
- net GPIO24: now also R14.1
- net GPIO25: now also R17.1
- net GPIO26: now also R29.1
- net GPIO27: now also R11.1
- net GPIO3: now also R5.1
- net GPIO4: now also R6.1
- net GPIO5: now also R23.1
- net GPIO6: now also R24.1
- net GPIO7: now also R20.1
- net GPIO8: now also R19.1
- net GPIO9: now also R16.1
- net ID_SC: now also R22.1, R32.1, U3.6 (SCL)
- net ID_SD: now also R21.1, R33.1, U3.5 (SDA)
- net LED_B: now also R1.2, U1.21 (PB13); no longer R3.2, U1.19 (PB11)
- net LED_R: now also R3.2, U1.19 (PB11); no longer R1.2, U1.21 (PB13)
- net PGPIO10: now also R15.2
- net PGPIO11: now also R18.2
- net PGPIO12: now also R25.2
- net PGPIO13: now also R26.2
- net PGPIO14: now also R7.2
- net PGPIO15: now also R8.2
- net PGPIO16: now also R28.2
- net PGPIO17: now also R9.2
- net PGPIO18: now also R10.2
- net PGPIO19: now also R27.2
- net PGPIO2: now also R4.2
- net PGPIO20: now also R30.2
- net PGPIO21: now also R31.2
- net PGPIO22: now also R12.2
- net PGPIO23: now also R13.2
- net PGPIO24: now also R14.2
- net PGPIO25: now also R17.2
- net PGPIO26: now also R29.2
- net PGPIO27: now also R11.2
- net PGPIO3: now also R5.2
- net PGPIO4: now also R6.2
- net PGPIO5: now also R23.2
- net PGPIO6: now also R24.2
- net PGPIO7: now also R20.2
- net PGPIO8: now also R19.2
- net PGPIO9: now also R16.2
- net PID_SC: now also R22.2
- net PID_SD: now also R21.2
- net VDD: now also D1.1 (A), JP6.1, JP7.1, R32.2, R33.2, U3.8 (VCC); no longer U2.5 (VOUT)
- net 3V3_IN: now reaches J1.1 (P1)
- net 3V3_IN: now also JP7.2
- net at R1.1: now also D1.2 (RK)
- net at R2.1: now also D1.3 (GK)
- net at R3.1: now also D1.4 (BK)
- new net 3V3_REG: JP6.2, U2.5 (VOUT)
Other:
- note added: "U2: AP2210K-3.3, alt: NJM2866F33-TE1, alt: LP2985\nResistor net: Bourns CAY16-221J4LF, is 3.2×1.6 mm\nCrystal: TSX-3225 38.4000MF10Z-AS3\nRGB LED: ASMB-MTB0-0A3A2 or CLMVB-FKA-CFHEHLCBB7a363\nPossible improvements:\n - Add ARM debug header\n - reset switch option\n - OSHW logo\n - Revision info on bottom side\n"
- note removed: "U2: AP2210K-3.3, alt: NJM2866F33-TE1, alt: LP2985\nOption: change VREG for 1.8V operation?\nResistor net: Bourns CAY16-221J4LF, is 3.2×1.6 mm\nCrystal: TSX-3225 38.4000MF10Z-AS3\nFIXME:\n - Add ARM debug header\n - reset switch option\n - Elemental logo\n - OSHW logo\n - Revision info on bottom side\n - Jumpers over resistor nets\n - 3V3 vreg bypass jumper\n - Isolate GND on bottom of U1 and add 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"
- moved on the sheet: C3

Commit message: Replace a couple of cap footprints
Parts:
- C1, C3, C5: footprint Capacitors_SMD:C_0603_HandSoldering -> c_local:C_0603_1608Metric_Pad0.84x1.00mm_HandSolder
Changed lines of the file:
@@
 F 0 "C3" H 3625 1700 50  0000 L CNN
 F 1 "2.2u" H 3625 1500 50  0000 L CNN
-F 2 "Capacitors_SMD:C_0603_HandSoldering" H 3638 1450 50  0001 C CNN
+F 2 "c_local:C_0603_1608Metric_Pad0.84x1.00mm_HandSolder" H 3638 1450 50  0001 C CNN
 F 3 "" H 3600 1600 50  0001 C CNN
 	1    3600 1600
@@
 F 0 "C1" H 1010 1920 50  0000 L CNN
 F 1 "1u" H 1010 1770 50  0000 L CNN
-F 2 "Capacitors_SMD:C_0603_HandSoldering" H 1000 1850 50  0001 C CNN
+F 2 "c_local:C_0603_1608Metric_Pad0.84x1.00mm_HandSolder" H 1000 1850 50  0001 C CNN
 F 3 "" H 1000 1850 50  0001 C CNN
 	1    1000 1850
@@
 F 0 "C5" H 1310 2220 50  0000 L CNN
 F 1 "DNP" H 1310 2070 50  0000 L CNN
-F 2 "Capacitors_SMD:C_0603_HandSoldering" H 1300 2150 50  0001 C CNN
+F 2 "c_local:C_0603_1608Metric_Pad0.84x1.00mm_HandSolder" H 1300 2150 50  0001 C CNN
 F 3 "" H 1300 2150 50  0001 C CNN
 	1    1300 2150

Commit message: Specify part numbers
Parts:
- D1: value LED_ARGB -> ASMB-MTB0-0A3A2
- U2: value LP2985LV -> AP2210K-3.3
- Y1: value 38.4 MHz -> TSX-3225 38.4000MF10Z-AS3
Other:
- note added: "U1: EFM32JG1B100*M32 (or same EFM32PG with Cortex-M4)\nU2: AP2210K-3.3, alt: NJM2866F33-TE1, alt: LP2985\nResistor net: Bourns CAY16-221J4LF, is 3.2×1.6 mm\nCrystal: TSX-3225 38.4000MF10Z-AS3\nRGB LED: ASMB-MTB0-0A3A2 or CLMVB-FKA-CFHEHLCBB7a363\n"
- note removed: "U2: AP2210K-3.3, alt: NJM2866F33-TE1, alt: LP2985\nResistor net: Bourns CAY16-221J4LF, is 3.2×1.6 mm\nCrystal: TSX-3225 38.4000MF10Z-AS3\nRGB LED: ASMB-MTB0-0A3A2 or CLMVB-FKA-CFHEHLCBB7a363\nPossible improvements:\n - Add ARM debug header\n - reset switch option\n - OSHW logo\n - Revision info on bottom side\n"
Changed lines of the file:
@@
 P 2100 1750
 F 0 "U2" H 2300 1300 50  0000 C CNN
-F 1 "LP2985LV" H 2100 2200 50  0000 C CNN
+F 1 "AP2210K-3.3" H 2100 2200 50  0000 C CNN
 F 2 "TO_SOT_Packages_SMD:SOT-23-5_HandSoldering" H 2100 1750 50  0001 C CNN
 F 3 "" H 2100 1750 50  0001 C CNN
@@
 	1    0    0    -1
 $EndComp
-Text Notes 3750 6700 0    60   ~ 0
-U2: AP2210K-3.3, alt: NJM2866F33-TE1, alt: LP2985\nResistor net: Bourns CAY16-221J4LF, is 3.2×1.6 mm\nCrystal:  TSX-3225 38.4000MF10Z-AS3\nRGB LED: ASMB-MTB0-0A3A2 or CLMVB-FKA-CFHEHLCBB7a363\nPossible improvements:\n  - Add ARM debug header\n  - reset switch option\n  - OSHW logo\n  - Revision info on bottom side\n
+Text Notes 3650 6000 0    60   ~ 0
+U1: EFM32JG1B100*M32 (or same EFM32PG with Cortex-M4)\nU2: AP2210K-3.3, alt: NJM2866F33-TE1, alt: LP2985\nResistor net: Bourns CAY16-221J4LF, is 3.2×1.6 mm\nCrystal:  TSX-3225 38.4000MF10Z-AS3\nRGB LED: ASMB-MTB0-0A3A2 or CLMVB-FKA-CFHEHLCBB7a363\n
 $Comp
 L +5V #PWR011
@@
 P 900 4850
 F 0 "Y1" H 1025 5050 50  0000 L CNN
-F 1 "38.4 MHz" H 1025 4975 50  0000 L CNN
+F 1 "TSX-3225 38.4000MF10Z-AS3" H 1025 4975 50  0000 L CNN
 F 2 "Crystals:Crystal_SMD_SeikoEpson_FA238-4pin_3.2x2.5mm_HandSoldering" H 900 4850 50  0001 C CNN
 F 3 "" H 900 4850 50  0001 C CNN
@@
 P 4700 4600
 F 0 "D1" H 4700 4970 50  0000 C CNN
-F 1 "LED_ARGB" H 4700 4250 50  0000 C CNN
+F 1 "ASMB-MTB0-0A3A2" H 4700 4250 50  0000 C CNN
 F 2 "led:LED_Avago_PLCC4_3.2x2.8mm_CW" H 4700 4550 50  0001 C CNN
 F 3 "" H 4700 4550 50  0001 C CNN

Commit message: Silk work
Parts:
- C2, C6, C7, C8, C9: footprint Capacitors_SMD:C_0603_HandSoldering -> c_local:C_0603_1608Metric_Pad0.84x1.00mm_HandSolder
Changed lines of the file:
@@
 F 0 "C2" H 1960 6820 50  0000 L CNN
 F 1 "0.1u" H 1960 6670 50  0000 L CNN
-F 2 "Capacitors_SMD:C_0603_HandSoldering" H 1950 6750 50  0001 C CNN
+F 2 "c_local:C_0603_1608Metric_Pad0.84x1.00mm_HandSolder" H 1950 6750 50  0001 C CNN
 F 3 "" H 1950 6750 50  0001 C CNN
 	1    1950 6750
@@
 F 0 "C9" H 3110 3620 50  0000 L CNN
 F 1 "1u" H 3110 3470 50  0000 L CNN
-F 2 "Capacitors_SMD:C_0603_HandSoldering" H 3100 3550 50  0001 C CNN
+F 2 "c_local:C_0603_1608Metric_Pad0.84x1.00mm_HandSolder" H 3100 3550 50  0001 C CNN
 F 3 "" H 3100 3550 50  0001 C CNN
 	1    3100 3550
@@
 F 0 "C6" H 1610 6820 50  0000 L CNN
 F 1 "0.1u" H 1610 6670 50  0000 L CNN
-F 2 "Capacitors_SMD:C_0603_HandSoldering" H 1600 6750 50  0001 C CNN
+F 2 "c_local:C_0603_1608Metric_Pad0.84x1.00mm_HandSolder" H 1600 6750 50  0001 C CNN
 F 3 "" H 1600 6750 50  0001 C CNN
 	1    1600 6750
@@
 F 0 "C7" H 2310 6820 50  0000 L CNN
 F 1 "10n" H 2310 6670 50  0000 L CNN
-F 2 "Capacitors_SMD:C_0603_HandSoldering" H 2300 6750 50  0001 C CNN
+F 2 "c_local:C_0603_1608Metric_Pad0.84x1.00mm_HandSolder" H 2300 6750 50  0001 C CNN
 F 3 "" H 2300 6750 50  0001 C CNN
 	1    2300 6750
@@
 F 0 "C8" H 2660 6820 50  0000 L CNN
 F 1 "10n" H 2660 6670 50  0000 L CNN
-F 2 "Capacitors_SMD:C_0603_HandSoldering" H 2650 6750 50  0001 C CNN
+F 2 "c_local:C_0603_1608Metric_Pad0.84x1.00mm_HandSolder" H 2650 6750 50  0001 C CNN
 F 3 "" H 2650 6750 50  0001 C CNN
 	1    2650 6750

Commit message: Change to TSSOP EEPROM, so it fits
Parts:
- added C10: 0.1u, c_local:C_0603_1608Metric_Pad0.84x1.00mm_HandSolder, symbol C_Small
- U3: value CAT24C32 -> CAT24C32Y; footprint Housings_SOIC:SOIC-8_3.9x4.9mm_Pitch1.27mm -> Housings_SSOP:TSSOP-8_4.4x3mm_Pitch0.65mm
Connections:
- net GND: now also C10.2
- net VDD: now also C10.1
